Commit message: restore capsule for pelvis

File: urdf/centauro_dagana_virtual_frame_capsule.urdf (robot description, URDF)
Before this commit: robot centauro, 64 links, 63 joints
Links:
- link pelvis: geometry collision cylinder length=0.38594139791384763 radius=0.213204; collision sphere radius=0.213204
